Commit message: Add State Interfaces for mimic joints (#14)
* Add State Interfaces for mimic joints

* Bugfixes

* removed double initialization

* Updated Readme

* added mimic joint to test robot xacro

* Bugfix Normal Joint Loading in Presence of Mimic Joints

* Updated Readme

File: dynamixel_ros_control/config/ros2_control_test_config.xacro (robot description, xacro)
@@ -23,4 +23,10 @@
                 <state_interface name="effort"/>
             </joint>
+            <joint name="mimic_joint">
+                <mimic>true</mimic>
+                <state_interface name="position"/>
+                <state_interface name="velocity"/>
+                <state_interface name="effort"/>
+            </joint>
             <transmission name="transmission1">
                 <plugin>transmission_interface/SimpleTransmission</plugin>

File: dynamixel_ros_control/config/test_robot.urdf.xacro (robot description, xacro)
@@ -9,4 +9,13 @@
     </joint>
     <link name="link_1"/>
+    <joint name="mimic_joint" type="continuous">
+      <parent link="link_1" />
+      <child link="link_2" />
+      <origin rpy="0 0 0" xyz="0 0.008 0.048" />
+      <axis xyz="1 0 0" />
+      <limit effort="1000" velocity="1.5" />
+      <mimic joint="joint_1" multiplier="2" offset="1" />
+    </joint>
+    <link name="link_2"/>
     <xacro:include filename="$(find dynamixel_ros_control)/config/ros2_control_test_config.xacro" />
     <xacro:ros2_control_test_config port_name="$(arg port_name)" baud_rate="$(arg baud_rate)" id="$(arg id)"/>

Commit message: updated function signature of on_init (#18)
* updated function signature of on_init

* applied updated pre-commits

File: dynamixel_ros_control/config/ros2_control_test_config.xacro (robot description, xacro)
@@ -1,41 +1,41 @@
-<?xml version="1.0"?>
+<?xml version="1.0" encoding="UTF-8"?>
 <robot xmlns:xacro="http://www.ros.org/wiki/xacro">
-    <xacro:macro name="ros2_control_test_config" params="port_name baud_rate id">
-        <ros2_control name="hardware_interface" type="system">
-            <hardware>
-                <plugin>dynamixel_ros_control/DynamixelHardwareInterface</plugin>
-                <param name="debug">true</param>
-                <param name="port_name">${port_name}</param>
-                <param name="baud_rate">${baud_rate}</param>
-                <param name="torque_on_startup">true</param>
-                <param name="torque_off_on_shutdown">true</param>
-                <param name="reboot_on_hardware_error">false</param>
-            </hardware>
-            <joint name="joint_1">
-                <param name="id">${id}</param>
-                <param name="position_control_mode">extended_position</param>
-                <param name="registers.velocity_limit">1.0</param>
-                <command_interface name="position"/>
-                <command_interface name="velocity"/>
-                <command_interface name="current"/>
-                <state_interface name="position"/>
-                <state_interface name="velocity"/>
-                <state_interface name="effort"/>
-            </joint>
-            <joint name="mimic_joint">
-                <mimic>true</mimic>
-                <state_interface name="position"/>
-                <state_interface name="velocity"/>
-                <state_interface name="effort"/>
-            </joint>
-            <transmission name="transmission1">
-                <plugin>transmission_interface/SimpleTransmission</plugin>
-                <actuator name="actuator_1" role="actuator_1"/>
-                <joint name="joint_1" role="joint_1">
-                    <mechanical_reduction>2.0</mechanical_reduction>
-                    <offset>0.0</offset>
-                </joint>
-            </transmission>
-        </ros2_control>
-    </xacro:macro>
+  <xacro:macro name="ros2_control_test_config" params="port_name baud_rate id">
+    <ros2_control name="hardware_interface" type="system">
+      <hardware>
+        <plugin>dynamixel_ros_control/DynamixelHardwareInterface</plugin>
+        <param name="debug">true</param>
+        <param name="port_name">${port_name}</param>
+        <param name="baud_rate">${baud_rate}</param>
+        <param name="torque_on_startup">true</param>
+        <param name="torque_off_on_shutdown">true</param>
+        <param name="reboot_on_hardware_error">false</param>
+      </hardware>
+      <joint name="joint_1">
+        <param name="id">${id}</param>
+        <param name="position_control_mode">extended_position</param>
+        <param name="registers.velocity_limit">1.0</param>
+        <command_interface name="position"/>
+        <command_interface name="velocity"/>
+        <command_interface name="current"/>
+        <state_interface name="position"/>
+        <state_interface name="velocity"/>
+        <state_interface name="effort"/>
+      </joint>
+      <joint name="mimic_joint">
+        <mimic>true</mimic>
+        <state_interface name="position"/>
+        <state_interface name="velocity"/>
+        <state_interface name="effort"/>
+      </joint>
+      <transmission name="transmission1">
+        <plugin>transmission_interface/SimpleTransmission</plugin>
+        <actuator name="actuator_1" role="actuator_1"/>
+        <joint name="joint_1" role="joint_1">
+          <mechanical_reduction>2.0</mechanical_reduction>
+          <offset>0.0</offset>
+        </joint>
+      </transmission>
+    </ros2_control>
+  </xacro:macro>
 </robot>

File: dynamixel_ros_control/config/test_robot.urdf.xacro (robot description, xacro)
@@ -1,22 +1,22 @@
-<?xml version="1.0"?>
+<?xml version="1.0" encoding="UTF-8"?>
 <robot xmlns:xacro="http://www.ros.org/wiki/xacro" name="test_robot">
-    <link name="base_link" />
-    <joint name="joint_1" type="continuous">
-        <parent link="base_link"/>
-        <child link="link_1"/>
-        <axis xyz="1 0 0" rpy="0 0 0" />
-        <limit effort="1000" velocity="1.5"/>
-    </joint>
-    <link name="link_1"/>
-    <joint name="mimic_joint" type="continuous">
-      <parent link="link_1" />
-      <child link="link_2" />
-      <origin rpy="0 0 0" xyz="0 0.008 0.048" />
-      <axis xyz="1 0 0" />
-      <limit effort="1000" velocity="1.5" />
-      <mimic joint="joint_1" multiplier="2" offset="1" />
-    </joint>
-    <link name="link_2"/>
-    <xacro:include filename="$(find dynamixel_ros_control)/config/ros2_control_test_config.xacro" />
-    <xacro:ros2_control_test_config port_name="$(arg port_name)" baud_rate="$(arg baud_rate)" id="$(arg id)"/>
+  <link name="base_link"/>
+  <joint name="joint_1" type="continuous">
+    <parent link="base_link"/>
+    <child link="link_1"/>
+    <axis xyz="1 0 0" rpy="0 0 0"/>
+    <limit effort="1000" velocity="1.5"/>
+  </joint>
+  <link name="link_1"/>
+  <joint name="mimic_joint" type="continuous">
+    <parent link="link_1"/>
+    <child link="link_2"/>
+    <origin rpy="0 0 0" xyz="0 0.008 0.048"/>
+    <axis xyz="1 0 0"/>
+    <limit effort="1000" velocity="1.5"/>
+    <mimic joint="joint_1" multiplier="2" offset="1"/>
+  </joint>
+  <link name="link_2"/>
+  <xacro:include filename="$(find dynamixel_ros_control)/config/ros2_control_test_config.xacro"/>
+  <xacro:ros2_control_test_config port_name="$(arg port_name)" baud_rate="$(arg baud_rate)" id="$(arg id)"/>
 </robot>
